File: High_Voltage_Power_Supply/_autosave-High_Voltage_Power_Supply.kicad_pcb (KiCad board)
At the start: 2 copper layers, 220 x 125 mm, 98 parts, among them J1 Conn_01x02_Female, J2 Conn_01x02_Female, J3 Conn_01x02_Female, J4 Conn_01x12_Female, Q1 Q_NMOS_GDS, Q2 Q_NMOS_GDS, Q3 Q_NMOS_GDS, Q4 Q_NIGBT_GCE, U1 LT3751-TSSOP, U10 ADR3412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

Commit message: updated BOM
Parts:
- moved C10 13.0 mm to (140.5, 46.5)
- moved C9 13.0 mm to (137.0, 46.5)
Changed lines of the file:
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@@
   )
   (module Capacitor_SMD:C_1210_3225Metric (layer F.Cu)
-    (at 153.5 46 90)
+    (at 140.5 46.5 90)
     (descr "Capacitor SMD 1210 (3225 Metric), square (rectangular) end terminal, IPC_7351 nominal, (Body size source: IPC-SM-782 page 76, https://www.pcb-3d.com/wordpress/wp-content/uploads/ipc-sm-782a_amendment_1_and_2.pdf), generated with kicad-footprint-generator")
     (tags capacitor)
@@
   )
   (module Capacitor_SMD:C_1210_3225Metric (layer F.Cu)
-    (at 150 46 90)
+    (at 137 46.5 90)
     (descr "Capacitor SMD 1210 (3225 Metric), square (rectangular) end terminal, IPC_7351 nominal, (Body size source: IPC-SM-782 page 76, https://www.pcb-3d.com/wordpress/wp-content/uploads/ipc-sm-782a_amendment_1_and_2.pdf), generated with kicad-footprint-generator")
     (tags capacitor)
